Commit message: Learning nodes and topics of ROS

File: differential_robot_185247iacb/urdf/differential_robot.urdf (robot description, URDF)
Before this commit: robot wroom_wroom, 6 links, 5 joints
Links:
- link base_link: mass None -> 0.1; geometry collision cylinder length=0.024 radius=0.0825; visual cylinder length=0.024 radius=0.0825
- link head: mass None -> 0.02; geometry collision box size=0.03 0.03 0.03; visual box size=0.03 0.03 0.03
- link left_wheel: mass None -> 0.015; geometry collision cylinder length=0.008 radius=0.035; visual cylinder length=0.008 radius=0.035
- link passive_wheel: mass None -> 0.02; geometry collision sphere radius=0.0075; visual sphere radius=0.0075
- link passive_wheel_holder: mass None -> 0.02; geometry collision cylinder length=0.0155 radius=0.0075; visual cylinder length=0.0155 radius=0.0075
- link right_wheel: mass None -> 0.015; geometry collision cylinder length=0.008 radius=0.035; visual cylinder length=0.008 radius=0.035
Joints:
- joint base_to_left_wheel: axis (none) -> 0 1 0; type fixed -> continuous
- joint base_to_right_wheel: axis (none) -> 0 1 0; type fixed -> continuous

Commit message: Making the earlier made robot move

File: differential_robot_185247iacb/urdf/differential_robot.urdf (robot description, URDF)
Before this commit: robot wroom_wroom, 6 links, 5 joints
Links:
- added link base_footprint
Joints:
- added joint base_footprint to base_link: type fixed, parent base_footprint, child base_link, origin xyz=0 0 0.035
